File: PCB/rd/rd.kicad_pcb (KiCad board)
At the start: 2 copper layers, 15 x 29.5 mm, 14 parts, among them U1 GL823K-HCY04

Commit message: routing
Parts:
- removed R2: 5.1k, easyeda2kicad:R0402
- USB1: value GT-USB-8016B -> U-USBAR04P-M001; footprint easyeda2kicad:USB-SMD_GT-USB-8016B -> easyeda2kicad:USB-SMD_KH-USB-AM-4P-CB
- moved LED1 12.2 mm to (72.6, 84.6), turned to 90 degrees
- moved R1 11.4 mm to (74.8, 83.7), turned to 90 degrees
- moved U1 2.78 mm to (81.7, 85.3)
- moved C1 2.78 mm to (85.2, 82.8)
- moved C2 2.78 mm to (85.0, 87.6)
- moved C3 2.78 mm to (86.5, 83.0)
- moved USB1 1.26 mm to (79.5, 78.1)
- moved R11 0.82 mm to (82.5, 89.8)
- moved Card1 0.39 mm to (80.0, 96.8)
- moved R9 0.35 mm to (79.4, 90.1)
Connections:
- USB1 pad 1: GND -> /VBUS
- USB1 pad 2: GND -> /D-
- USB1 pad 3: GND -> /D+
Routing:
- net /PMOS: track 0.00 -> 19.0 mm, vias 0 -> 4
- net /VDD: track 0.00 -> 18.8 mm, vias 0 -> 2
- net /VBUS: track 0.00 -> 13.3 mm
- net /LED: track 0.00 -> 11.6 mm, vias 0 -> 2
- net /D1: track 0.00 -> 11.1 mm
- net /D0: track 0.00 -> 7.84 mm
- net GND: track 0.00 -> 7.81 mm, vias 0 -> 2
- net /CLK: track 0.00 -> 5.90 mm
- net /CMD: track 0.00 -> 4.69 mm
- net /D2: track 0.00 -> 4.60 mm
- net /D3: track 0.00 -> 4.10 mm
- net /D+: track 0.00 -> 3.87 mm
- net /D-: track 0.00 -> 3.79 mm
- net Net-(LED1-A): track 0.00 -> 2.38 mm
- added copper zone on F.Cu, net GND
Other:
- board size 15 x 29.5 mm -> 18.5 x 32 mm

Commit message: regerb
Parts:
- moved USB1 0.55 mm to (80.0, 78.1)
Routing:
- net GND: track 7.81 -> 8.36 mm
Changed lines of the file:
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@@
 	(footprint "easyeda2kicad:USB-SMD_KH-USB-AM-4P-CB"
 		(layer "F.Cu")
-		(at 79.45 78.12 180)
+		(at 80 78.12 180)
 		(property "Reference" "USB1"
 			(at 0 -5.125 0)
@@
 	)
 	(segment
+		(start 81.8 80.79)
+		(end 81.209999 80.79)
+		(width 0.2)
+		(layer "F.Cu")
+		(net "GND")
+	)
+	(segment
 		(start 79.47 87.91)
 		(end 78.31 87.91)
@@
 	)
 	(segment
-		(start 80.74 82.61)
-		(end 80.74 81.26)
+		(start 80.74 81.259999)
+		(end 80.74 82.61)
+		(width 0.2)
+		(layer "F.Cu")
+		(net "GND")
+	)
+	(segment
+		(start 81.209999 80.79)
+		(end 80.74 81.259999)
 		(width 0.2)
 		(layer "F.Cu")
@@
 	)
 	(segment
-		(start 82.76 79.24)
-		(end 82.95 79.24)
+		(start 83.35 79.24)
+		(end 81.8 80.79)
 		(width 0.2)
 		(layer "F.Cu")
@@
 	)
 	(segment
-		(start 80.74 81.26)
-		(end 82.76 79.24)
+		(start 83.5 79.24)
+		(end 83.35 79.24)
 		(width 0.2)
 		(layer "F.Cu")
@@
 	)
 	(segment
-		(start 83.91 81.3025)
-		(end 83.91 82.61)
-		(width 0.4)
-		(layer "F.Cu")
-		(net "/VDD")
-	)
-	(segment
 		(start 84.11 82.41)
 		(end 85.25 82.41)
@@
 	)
 	(segment
+		(start 81.37 81.337106)
+		(end 81.417106 81.29)
+		(width 0.4)
+		(layer "F.Cu")
+		(net "/VDD")
+	)
+	(segment
 		(start 85.25 82.41)
 		(end 86.34 82.41)
@@
 	)
 	(segment
-		(start 81.527106 81.18)
-		(end 83.7875 81.18)
-		(width 0.4)
-		(layer "F.Cu")
-		(net "/VDD")
-	)
-	(segment
 		(start 83.91 82.61)
 		(end 84.11 82.41)
@@
 	)
 	(segment
-		(start 81.37 81.337106)
-		(end 81.527106 81.18)
+		(start 83.7875 81.18)
+		(end 83.91 81.3025)
 		(width 0.4)
 		(layer "F.Cu")
@@
 	)
 	(segment
+		(start 81.37 82.61)
+		(end 81.37 81.337106)
+		(width 0.4)
+		(layer "F.Cu")
+		(net "/VDD")
+	)
+	(segment
 		(start 81.37 81.38)
 		(end 81.5 81.25)
 		(width 0.2)
-		(layer "F.Cu")
-		(net "/VDD")
-	)
-	(segment
-		(start 83.7875 81.18)
-		(end 83.91 81.3025)
-		(width 0.4)
 		(layer "F.Cu")
 		(net "/VDD")
@@
 	)
 	(segment
-		(start 81.37 82.61)
-		(end 81.37 81.337106)
+		(start 82.117106 81.18)
+		(end 83.7875 81.18)
+		(width 0.4)
+		(layer "F.Cu")
+		(net "/VDD")
+	)
+	(segment
+		(start 81.417106 81.29)
+		(end 82.007107 81.29)
+		(width 0.4)
+		(layer "F.Cu")
+		(net "/VDD")
+	)
+	(segment
+		(start 82.007107 81.29)
+		(end 82.117106 81.18)
+		(width 0.4)
+		(layer "F.Cu")
+		(net "/VDD")
+	)
+	(segment
+		(start 83.91 81.3025)
+		(end 83.91 82.61)
 		(width 0.4)
 		(layer "F.Cu")
@@
 	)
 	(segment
-		(start 78.45 79.99)
-		(end 79.225 80.765)
+		(start 79 79.24)
+		(end 79 82.14)
 		(width 0.2)
 		(layer "F.Cu")
@@
 	)
 	(segment
-		(start 79.225 80.765)
-		(end 79.225 82.365)
+		(start 79 82.14)
+		(end 79.47 82.61)
 		(width 0.2)
 		(layer "F.Cu")
@@
 	)
 	(segment
-		(start 78.45 79.24)
-		(end 78.45 79.99)
-		(width 0.2)
-		(layer "F.Cu")
-		(net "/D-")
-	)
-	(segment
-		(start 79.675 80.765)
-		(end 79.675 81.409497)
+		(start 80.1 80.14)
+		(end 81 79.24)
 		(width 0.2)
 		(layer "F.Cu")
@@
 	)
 	(segment
-		(start 80.45 79.99)
-		(end 79.675 80.765)
+		(start 80.1 82.61)
+		(end 80.1 80.14)
 		(width 0.2)
 		(layer "F.Cu")
@@
 	)
 	(segment
-		(start 80.45 79.24)
-		(end 80.45 79.99)
-		(width 0.2)
-		(layer "F.Cu")
-		(net "/D+")
-	)
-	(segment
-		(start 79.675 81.409497)
-		(end 80.1 81.834497)
-		(width 0.2)
-		(layer "F.Cu")
-		(net "/D+")
-	)
-	(segment
-		(start 80.1 81.834497)
-		(end 80.1 82.61)
-		(width 0.2)
-		(layer "F.Cu")
-		(net "/D+")
-	)
-	(segment
-		(start 75.95 80.89)
-		(end 75.95 79.24)
+		(start 76.73 81.67)
+		(end 76.73 79.47)
 		(width 0.4)
 		(layer "F.Cu")
@@
 	)
 	(segment
-		(start 78.9775 83.9175)
-		(end 75.95 80.89)
+		(start 76.73 79.47)
+		(end 76.5 79.24)
 		(width 0.4)
 		(layer "F.Cu")
@@
 		(width 0.4)
 		(layer "F.Cu")
+		(net "/VBUS")
+	)
+	(segment
+		(start 78.9775 83.9175)
+		(end 76.73 81.67)
+		(width 0.4)
+		(layer "F.Cu")

Commit message: ye
Parts:
- moved LED1 0.79 mm to (72.6, 85.3)
- moved R1 0.59 mm to (75.3, 83.9)
Other:
- outline, holes or cut-outs redrawn
- board text added: "rd"
Changed lines of the file:
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@@
 	(footprint "easyeda2kicad:LED0805-R-RD"
 		(layer "F.Cu")
-		(at 72.625 84.555 90)
+		(at 72.625 85.35 90)
 		(descr "0805")
 		(property "Reference" "LED1"
@@
 	(footprint "easyeda2kicad:R0402"
 		(layer "F.Cu")
-		(at 74.75 83.68 90)
+		(at 75.3 83.9 90)
 		(property "Reference" "R1"
 			(at 0 -4 90)
@@
 		(layer "Edge.Cuts")
 	)
+	(gr_circle
+		(center 73.5 81)
+		(end 75.5 81)
+		(stroke
+			(width 0.05)
+			(type solid)
+		)
+		(fill no)
+		(layer "Edge.Cuts")
+	)
+	(gr_text "rd"
+		(at 72 103.9 270)
+		(layer "B.SilkS")
+		(effects
+			(font
+				(face "TX-02-Data")
+				(size 13 13)
+				(thickness 0.1)
+			)
+			(justify left bottom mirror)
+		)
+		(render_cache "rd" 270
+			(polygon
+				(pts
+					(xy 74.21 100.69706) (xy 74.21 99.296022) (xy 77.978911 99.296022) (xy 79.065641 99.26824) (xy 79.961812 99.175369)
+					(xy 80.479138 99.065488) (xy 80.918658 98.91286) (xy 81.230884 98.748702) (xy 81.495629 98.54846)
+					(xy 81.873422 98.069446) (xy 82.124503 97.413807) (xy 82.266513 96.453968) (xy 82.293949 95.583469)
+					(xy 82.271128 94.937027) (xy 82.166149 94.236409) (xy 83.567981 94.236409) (xy 83.651571 95.200992)
+					(xy 83.662227 96.285597) (xy 83.659267 96.474895) (xy 83.639495 97.251652) (xy 83.572064 97.829304)
+					(xy 83.419607 98.265251) (xy 83.144761 98.616897) (xy 82.56971 99.026802) (xy 81.656536 99.514314)
+					(xy 81.656536 99.6056) (xy 83.64101 99.441285) (xy 83.64101 100.69706)
+				)
+			)
+			(polygon
+				(pts
+					(xy 87.57106 83.763154) (xy 87.57106 85.183243) (xy 82.59162 85.164986) (xy 82.59162 85.255478)
+					(xy 83.014987 85.448335) (xy 83.331739 85.67785) (xy 83.492544 85.868165) (xy 83.615251 86.096966)
+					(xy 83.764839 86.715154) (xy 83.811674 87.712255) (xy 83.784107 88.592361) (xy 83.692744 89.336741)
+					(xy 83.580576 89.793136) (xy 83.424038 90.18873) (xy 83.251093 90.482043) (xy 83.039072 90.735966)
+					(xy 82.515893 91.119472) (xy 81.781861 91.394957) (xy 80.697878 91.574385) (xy 78.918757 91.643893)
+					(xy 77.705595 91.61612) (xy 76.701129 91.523311) (xy 76.11748 91.413217) (xy 75.619647 91.260226)
+					(xy 75.266036 91.096545) (xy 74.964397 90.897029) (xy 74.730379 90.680075) (xy 74.53453 90.42851)
+					(xy 74.244515 89.806447) (xy 74.06629 88.927994) (xy 74.006789 87.694792) (xy 74.008689 87.64002)
+					(xy 75.334799 87.64002) (xy 75.362735 88.305964) (xy 75.456685 88.85223) (xy 75.567902 89.164847)
+					(xy 75.722752 89.429111) (xy 75.898841 89.624234) (xy 76.115883 89.787087) (xy 76.700424 90.029357)
+					(xy 77.627664 90.179261) (xy 78.908438 90.223804) (xy 79.973845 90.195615) (xy 80.81463 90.099895)
+					(xy 81.254098 89.992908) (xy 81.614718 89.845299) (xy 81.859197 89.68841) (xy 82.057737 89.497583)
+					(xy 82.323111 89.029462) (xy 82.469183 88.345342) (xy 82.501128 87.64002) (xy 82.473163 86.980114)
+					(xy 82.379009 86.439774) (xy 82.267811 86.131843) (xy 82.113003 85.871825) (xy 81.936611 85.679739)
+					(xy 81.719107 85.519649) (xy 81.130419 85.28135) (xy 80.190322 85.134509) (xy 78.908438 85.091957)
+					(xy 77.830998 85.120364) (xy 76.984859 85.21761) (xy 76.551632 85.324758) (xy 76.1967 85.472525)
+					(xy 75.956785 85.62943) (xy 75.762354 85.820339) (xy 75.503193 86.290296) (xy 75.362605 86.981451)
+					(xy 75.334799 87.64002) (xy 74.008689 87.64002) (xy 74.036502 86.838266) (xy 74.142886 86.21227)
+					(xy 74.251265 85.931073) (xy 74.400095 85.699983) (xy 74.796126 85.370263) (xy 75.22605 85.164986)
+					(xy 75.245894 85.0737) (xy 74.21 85.0737) (xy 74.21 83.744897)
+				)
+			)
+		)
+	)
 	(segment
 		(start 81.8 80.79)
@@
 	)
 	(segment
-		(start 74.75 83.25)
-		(end 76.5 83.25)
-		(width 0.2)
-		(layer "F.Cu")
-		(net "/VDD")
-	)
-	(segment
 		(start 83.7875 81.18)
 		(end 83.91 81.3025)
@@
 	)
 	(segment
+		(start 75.52 83.25)
+		(end 76.5 83.25)
+		(width 0.2)
+		(layer "F.Cu")
+		(net "/VDD")
+	)
+	(segment
 		(start 86.34 82.41)
 		(end 86.5 82.57)
@@
 	)
 	(segment
+		(start 75.3 83.47)
+		(end 75.52 83.25)
+		(width 0.2)
+		(layer "F.Cu")
+		(net "/VDD")
+	)
+	(segment
 		(start 82.117106 81.18)
 		(end 83.7875 81.18)
@@
 	)
 	(segment
-		(start 73.23 84.11)
-		(end 74.75 84.11)
+		(start 72.655 84.33)
+		(end 72.625 84.3)
 		(width 0.2)
 		(layer "F.Cu")
@@
 	)
 	(segment
-		(start 72.625 83.505)
-		(end 73.23 84.11)
+		(start 75.3 84.33)
+		(end 72.655 84.33)
 		(width 0.2)
 		(layer "F.Cu")
@@
 	)
 	(segment
-		(start 72.73 85.5)
-		(end 72.625 85.605)
+		(start 82.01 84.24)
+		(end 82 84.25)
 		(width 0.2)
 		(layer "F.Cu")
@@
 	)
 	(segment
-		(start 82.01 84.24)
-		(end 82 84.25)
+		(start 74.5 85.5)
+		(end 73.6 86.4)
 		(width 0.2)
 		(layer "F.Cu")
@@
 	)
 	(segment
-		(start 74.5 85.5)
-		(end 72.73 85.5)
+		(start 73.6 86.4)
+		(end 72.625 86.4)
 		(width 0.2)
 		(layer "F.Cu")
