File: PCB/rd/rd.kicad_sch (KiCad schematic)
At the start: 14 parts, among them U1 GL823K-HCY04

Commit message: routing
Parts:
- removed R2: 5.1k, easyeda2kicad:R0402, symbol lcsc:0402WGF5101TCE
- removed USB1: GT-USB-8016B, easyeda2kicad:USB-SMD_GT-USB-8016B, symbol lcsc:GT-USB-8016B
- added USB1: U-USBAR04P-M001, easyeda2kicad:USB-SMD_KH-USB-AM-4P-CB, symbol lcsc:U-USBAR04P-M001
Connections:
- net D+: now also USB1.3 (D+)
- net D-: now also USB1.2 (D-)
- net GND: now also USB1.4 (GND), USB1.5 (EH), USB1.6 (EH)
- net VBUS: now also USB1.1 (VCC)
- no-connect marks 7 -> 2

Commit message: emergency 47uF addition
Parts:
- removed C2: 100nF, easyeda2kicad:C0402, symbol lcsc:CL05B104KO5NNNC
- added C4: 47uF, easyeda2kicad:C0805, symbol lcsc:CL21A476MQYNNNE
Connections:
- net GND: now also C4.1
- net PMOS: now also C4.2
Changed lines of the file:
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@@
+	(wire
+		(pts
+			(xy 223.52 26.67) (xy 223.52 25.4)
+		)
+		(stroke
+			(width 0)
+			(type default)
+		)
+	)
 	(wire
 		(pts
@@
 	(wire
 		(pts
-			(xy 143.51 35.56) (xy 151.13 35.56)
+			(xy 209.55 26.67) (xy 223.52 26.67)
 		)
 		(stroke
@@
 	(wire
 		(pts
-			(xy 177.8 60.96) (xy 175.26 60.96)
+			(xy 143.51 35.56) (xy 151.13 35.56)
 		)
 		(stroke
@@
 	(wire
 		(pts
-			(xy 167.64 35.56) (xy 175.26 35.56)
+			(xy 177.8 60.96) (xy 175.26 60.96)
 		)
 		(stroke
@@
 	(wire
 		(pts
-			(xy 143.51 58.42) (xy 177.8 58.42)
+			(xy 167.64 35.56) (xy 175.26 35.56)
 		)
 		(stroke
@@
 	(wire
 		(pts
-			(xy 198.12 35.56) (xy 200.66 35.56)
+			(xy 143.51 58.42) (xy 177.8 58.42)
 		)
 		(stroke
@@
 	(wire
 		(pts
-			(xy 158.75 50.8) (xy 177.8 50.8)
+			(xy 198.12 35.56) (xy 200.66 35.56)
 		)
 		(stroke
@@
 	(wire
 		(pts
-			(xy 167.64 45.72) (xy 167.64 48.26)
+			(xy 158.75 50.8) (xy 177.8 50.8)
 		)
 		(stroke
@@
 	(wire
 		(pts
+			(xy 167.64 45.72) (xy 167.64 48.26)
+		)
+		(stroke
+			(width 0)
+			(type default)
+		)
+	)
+	(wire
+		(pts
 			(xy 158.75 35.56) (xy 167.64 35.56)
+		)
+		(stroke
+			(width 0)
+			(type default)
+		)
+	)
+	(wire
+		(pts
+			(xy 209.55 34.29) (xy 223.52 34.29)
+		)
+		(stroke
+			(width 0)
+			(type default)
+		)
+	)
+	(wire
+		(pts
+			(xy 223.52 34.29) (xy 223.52 35.56)
 		)
 		(stroke
@@
 	)
 	(symbol
-		(lib_id "lcsc:CL05B104KO5NNNC")
-		(at 223.52 30.48 90)
+		(lib_id "lcsc:CL21A476MQYNNNE")
+		(at 209.55 30.48 90)
 		(unit 1)
 		(body_style 1)
@@
 		(dnp no)
 		(fields_autoplaced yes)
-		(property "Reference" "C2"
-			(at 227.33 29.2099 90)
+		(property "Reference" "C4"
+			(at 213.36 29.2099 90)
 			(show_name no)
 			(do_not_autoplace no)
@@
 			)
 		)
-		(property "Value" "100nF"
-			(at 227.33 31.7499 90)
+		(property "Value" "47uF"
+			(at 213.36 31.7499 90)
 			(show_name no)
 			(do_not_autoplace no)
@@
 			)
 		)
-		(property "Footprint" "easyeda2kicad:C0402"
-			(at 231.14 30.48 0)
-			(hide yes)
-			(show_name no)
-			(do_not_autoplace no)
-			(effects
-				(font
-					(size 1.27 1.27)
-				)
-			)
-		)
-		(property "Datasheet" "https://lcsc.com/product-detail/Multilayer-Ceramic-Capacitors-MLCC-SMD-SMT_SAMSUNG_CL05B104KO5NNNC_100nF-104-10-16V_C1525.html"
-			(at 233.68 30.48 0)
-			(hide yes)
-			(show_name no)
-			(do_not_autoplace no)
-			(effects
-				(font
-					(size 1.27 1.27)
-				)
-			)
-		)
-		(property "Description" "100nF (104) ±10% 16V"
-			(at 223.52 30.48 0)
+		(property "Footprint" "easyeda2kicad:C0805"
+			(at 217.17 30.48 0)
+			(hide yes)
+			(show_name no)
+			(do_not_autoplace no)
+			(effects
+				(font
+					(size 1.27 1.27)
+				)
+			)
+		)
+		(property "Datasheet" "https://lcsc.com/product-detail/Multilayer-Ceramic-Capacitors-MLCC-SMD-SMT_SAMSUNG_CL21A476MQYNNNE_47uF-476-20-6-3V_C16780.html"
+			(at 219.71 30.48 0)
+			(hide yes)
+			(show_name no)
+			(do_not_autoplace no)
+			(effects
+				(font
+					(size 1.27 1.27)
+				)
+			)
+		)
+		(property "Description" "47uF (476) ±20% 6.3V"
+			(at 209.55 30.48 0)
 			(hide yes)
 			(show_name no)
@@
 		)
 		(property "Manufacturer" "SAMSUNG(三星)"
-			(at 236.22 30.48 0)
-			(hide yes)
-			(show_name no)
-			(do_not_autoplace no)
-			(effects
-				(font
-					(size 1.27 1.27)
-				)
-			)
-		)
-		(property "MPN" "CL05B104KO5NNNC"
-			(at 238.76 30.48 0)
-			(hide yes)
-			(show_name no)
-			(do_not_autoplace no)
-			(effects
-				(font
-					(size 1.27 1.27)
-				)
-			)
-		)
-		(property "LCSC Part" "C1525"
-			(at 241.3 30.48 0)
-			(hide yes)
-			(show_name no)
-			(do_not_autoplace no)
-			(effects
-				(font
-					(size 1.27 1.27)
-				)
-			)
+			(at 222.25 30.48 0)
+			(hide yes)
+			(show_name no)
+			(do_not_autoplace no)
+			(effects
+				(font
+					(size 1.27 1.27)
+				)
+			)
+		)
+		(property "MPN" "CL21A476MQYNNNE"
+			(at 224.79 30.48 0)
+			(hide yes)
+			(show_name no)
+			(do_not_autoplace no)
+			(effects
+				(font
+					(size 1.27 1.27)
+				)
+			)
+		)
+		(property "LCSC Part" "C16780"
+			(at 227.33 30.48 0)
+			(hide yes)
+			(show_name no)
+			(do_not_autoplace no)
+			(effects
+				(font
+					(size 1.27 1.27)
+				)
+			)
+		)
+		(pin "1"
 		)
 		(pin "2"
-		)
-		(pin "1"
 		)
 		(instances
 			(project "rd"
 				(path "/dbc6aea7-bd01-4206-baa9-133a282a0cbe"
-					(reference "C2")
+					(reference "C4")
 					(unit 1)
 				)
